Commit message: Modificacion el los marcos de referencia del robot

File: scora_ind/urdf/scora.urdf (robot description, URDF)
Before this commit: robot scora_ind, 12 links, 11 joints
Links:
- link Light_alarm: mass 0.072255 -> 0.0722547774929001
- link link2_bottom: mass 1.9512 -> 1.95123434278269; geometry collision mesh filename=package://scora_ind/link2_bottom.STL; visual mesh filename=package://scora_ind/link2_bottom.STL
- link link2_top: mass 3.9231 -> 3.92307386569457; geometry collision mesh filename=package://scora_ind/link2_top.STL; visual mesh filename=package://scora_ind/link2_top.STL
- link link_4: mass 0.45456 -> 0.53644; geometry collision mesh filename=package://scora_ind/link_4.STL; visual mesh filename=package://scora_ind/link_4.STL
- link link_top: mass 2.4093 -> 2.409257353011
Joints:
- joint gripper_left_to_link_4: origin xyz=-0.029935 -0.11 0 rpy=0 0 0 -> xyz=-0.04 4.2729E-05 0 rpy=1.5708 0 0
- joint gripper_right_to_link_4: origin xyz=0.020065 -0.11 0 rpy=3.1416 0 3.1416 -> xyz=0.04 -4.8156E-05 0 rpy=1.5708 0 -3.1416
- joint link2_bottom_to_link_2: origin xyz=0.115 0 -0.275 rpy=1.5708 0 3.1416 -> xyz=0.115 0 -0.13 rpy=1.5708 0 -3.1416
- joint link2_top_to_link_2: origin xyz=0.115 0 -0.145 rpy=1.5708 0 0 -> xyz=0.115 0 0 rpy=1.5708 0 0
- joint link_1_to_base_link: origin xyz=-0.035098 -0.14087 0.733 rpy=0 0 3.1354 -> xyz=-0.0055 0 0.588 rpy=0 0 -0.0062122
- joint link_2_to_link_1: origin xyz=0.27 0 0 rpy=0 0 -0.010618 -> xyz=0.27 0 0 rpy=0 0 0
- joint link_3_to_link_2: origin xyz=0.23 0 -0.275 rpy=0 0 0.01683 -> xyz=0.23 0 0 rpy=0 0 0
- joint link_4_to_link_3: axis 0 1 0 -> 0 0 1; origin xyz=0 0 -0.10799 rpy=1.5708 0 0.26415 -> xyz=0 0 -0.3478 rpy=0 0 0
- joint link_top_to_link_1: origin xyz=0.135 0 0.032 rpy=1.5708 0 3.1416 -> xyz=0.135 0 0.177 rpy=1.5708 0 -3.1416

File: scora_ind/urdf/scora_Joint_trajectory_controller.urdf (robot description, URDF)
Before this commit: robot scora_ind, 12 links, 11 joints
Links:
- link Light_alarm: mass 0.072255 -> 0.0722547774929001
- link link2_bottom: mass 1.9512 -> 1.95123434278269; geometry collision mesh filename=/home/smr/ros2_ws/src/scora-er_14/scora_ind/meshes/link2_bo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; visual mesh filename=/home/smr/ros2_ws/src/scora-er_14/scora_ind/meshes/link2_bo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
- link link2_top: mass 3.9231 -> 3.92307386569457; geometry collision mesh filename=/home/smr/ros2_ws/src/scora-er_14/scora_ind/meshes/link2_to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; visual mesh filename=/home/smr/ros2_ws/src/scora-er_14/scora_ind/meshes/link2_to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
- link link_4: mass 0.45456 -> 0.53644; geometry collision mesh filename=/home/smr/ros2_ws/src/scora-er_14/scora_ind/meshes/link_4.S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; visual mesh filename=/home/smr/ros2_ws/src/scora-er_14/scora_ind/meshes/link_4.S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
- link link_top: mass 2.4093 -> 2.409257353011
Joints:
- joint gripper_left_to_link_4: limit lower=0 upper=0.03 effort=1000 velocity=0.5 -> lower=0 upper=0.027 effort=1000 velocity=0.5; origin xyz=-0.029935 -0.11 0 rpy=0 0 0 -> xyz=-0.04 4.2729E-05 0 rpy=1.5708 0 0
- joint gripper_right_to_link_4: limit lower=0 upper=0.03 effort=1000 velocity=0.5 -> lower=0 upper=0.027 effort=1000 velocity=0.5; origin xyz=0.020065 -0.11 0 rpy=3.1416 0 3.1416 -> xyz=0.04 -4.8156E-05 0 rpy=1.5708 0 -3.1416
- joint link2_bottom_to_link_2: origin xyz=0.115 0 -0.275 rpy=1.5708 0 3.1416 -> xyz=0.115 0 -0.13 rpy=1.5708 0 -3.1416
- joint link2_top_to_link_2: origin xyz=0.115 0 -0.145 rpy=1.5708 0 0 -> xyz=0.115 0 0 rpy=1.5708 0 0
- joint link_1_to_base_link: limit lower=-2.5 upper=2.5 effort=1000 velocity=0.5 -> lower=-2.125 upper=2.125 effort=1000 velocity=0.5; origin xyz=-0.035098 -0.14087 0.733 rpy=0 0 3.1354 -> xyz=-0.0055 0 0.588 rpy=0 0 -0.0062122
- joint link_2_to_link_1: limit lower=-2.5 upper=2.5 effort=1000 velocity=0.5 -> lower=-2 upper=2 effort=1000 velocity=0.5; origin xyz=0.27 0 0 rpy=0 0 -0.010618 -> xyz=0.27 0 0 rpy=0 0 0
- joint link_3_to_link_2: limit lower=-0.15 upper=0 effort=1000 velocity=0.5 -> lower=-0.12 upper=0 effort=1000 velocity=0.5; origin xyz=0.23 0 -0.275 rpy=0 0 0.01683 -> xyz=0.23 0 0 rpy=0 0 0
- joint link_4_to_link_3: axis 0 1 0 -> 0 0 1; limit lower=0 upper=5 effort=1000 velocity=0.5 -> lower=0 upper=10 effort=1000 velocity=0.5; origin xyz=0 0 -0.10799 rpy=1.5708 0 0.26415 -> xyz=0 0 -0.3478 rpy=0 0 0
- joint link_top_to_link_1: origin xyz=0.135 0 0.032 rpy=1.5708 0 3.1416 -> xyz=0.135 0 0.177 rpy=1.5708 0 -3.1416

File: scora_ind/urdf/scora_gazebo.urdf (robot description, URDF)
Before this commit: robot scora_ind, 12 links, 11 joints
Links:
- link Light_alarm: mass 0.072255 -> 0.0722547774929001
- link link2_bottom: mass 1.9512 -> 1.95123434278269; geometry collision mesh filename=/home/smr/ros2_ws/src/scora-er_14/scora_ind/meshes/link2_bo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; visual mesh filename=/home/smr/ros2_ws/src/scora-er_14/scora_ind/meshes/link2_bo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
- link link2_top: mass 3.9231 -> 3.92307386569457; geometry collision mesh filename=/home/smr/ros2_ws/src/scora-er_14/scora_ind/meshes/link2_to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; visual mesh filename=/home/smr/ros2_ws/src/scora-er_14/scora_ind/meshes/link2_to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
- link link_4: mass 0.45456 -> 0.53644; geometry collision mesh filename=/home/smr/ros2_ws/src/scora-er_14/scora_ind/meshes/link_4.S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; visual mesh filename=/home/smr/ros2_ws/src/scora-er_14/scora_ind/meshes/link_4.S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
- link link_top: mass 2.4093 -> 2.409257353011
Joints:
- joint gripper_left_to_link_4: origin xyz=-0.029935 -0.11 0 rpy=0 0 0 -> xyz=-0.04 4.2729E-05 0 rpy=1.5708 0 0
- joint gripper_right_to_link_4: origin xyz=0.020065 -0.11 0 rpy=3.1416 0 3.1416 -> xyz=0.04 -4.8156E-05 0 rpy=1.5708 0 -3.1416
- joint link2_bottom_to_link_2: origin xyz=0.115 0 -0.275 rpy=1.5708 0 3.1416 -> xyz=0.115 0 -0.13 rpy=1.5708 0 -3.1416
- joint link2_top_to_link_2: origin xyz=0.115 0 -0.145 rpy=1.5708 0 0 -> xyz=0.115 0 0 rpy=1.5708 0 0
- joint link_1_to_base_link: origin xyz=-0.035098 -0.14087 0.733 rpy=0 0 3.1354 -> xyz=-0.0055 0 0.588 rpy=0 0 -0.0062122
- joint link_2_to_link_1: origin xyz=0.27 0 0 rpy=0 0 -0.010618 -> xyz=0.27 0 0 rpy=0 0 0
- joint link_3_to_link_2: origin xyz=0.23 0 -0.275 rpy=0 0 0.01683 -> xyz=0.23 0 0 rpy=0 0 0
- joint link_4_to_link_3: axis 0 1 0 -> 0 0 1; origin xyz=0 0 -0.10799 rpy=1.5708 0 0.26415 -> xyz=0 0 -0.3478 rpy=0 0 0
- joint link_top_to_link_1: origin xyz=0.135 0 0.032 rpy=1.5708 0 3.1416 -> xyz=0.135 0 0.177 rpy=1.5708 0 -3.1416
