Commit message: Mejoras en la interfaz

File: scora_ind/urdf/scora_Joint_trajectory_controller.urdf (robot description, URDF)
Before this commit: robot scora_ind, 12 links, 11 joints
Links:
- link Light_alarm: geometry collision mesh filename=/home/celdamanufactura/ros2_ws/src/scora-er_14/scora_ind/me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; visual mesh filename=/home/celdamanufactura/ros2_ws/src/scora-er_14/scora_ind/me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
- link base_link: geometry collision mesh filename=/home/celdamanufactura/ros2_ws/src/scora-er_14/scora_ind/me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; visual mesh filename=/home/celdamanufactura/ros2_ws/src/scora-er_14/scora_ind/me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
- link gripper_left: geometry collision mesh filename=/home/celdamanufactura/ros2_ws/src/scora-er_14/scora_ind/me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; visual mesh filename=/home/celdamanufactura/ros2_ws/src/scora-er_14/scora_ind/me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
- link gripper_right: geometry collision mesh filename=/home/celdamanufactura/ros2_ws/src/scora-er_14/scora_ind/me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; visual mesh filename=/home/celdamanufactura/ros2_ws/src/scora-er_14/scora_ind/me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
- link link2_bottom: geometry collision mesh filename=/home/celdamanufactura/ros2_ws/src/scora-er_14/scora_ind/me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; visual mesh filename=/home/celdamanufactura/ros2_ws/src/scora-er_14/scora_ind/me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
- link link2_top: geometry collision mesh filename=/home/celdamanufactura/ros2_ws/src/scora-er_14/scora_ind/me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; visual mesh filename=/home/celdamanufactura/ros2_ws/src/scora-er_14/scora_ind/me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
- link link_1: geometry collision mesh filename=/home/celdamanufactura/ros2_ws/src/scora-er_14/scora_ind/me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; visual mesh filename=/home/celdamanufactura/ros2_ws/src/scora-er_14/scora_ind/me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
- link link_2: geometry collision mesh filename=/home/celdamanufactura/ros2_ws/src/scora-er_14/scora_ind/me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; visual mesh filename=/home/celdamanufactura/ros2_ws/src/scora-er_14/scora_ind/me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
- link link_3: geometry collision mesh filename=/home/celdamanufactura/ros2_ws/src/scora-er_14/scora_ind/me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; visual mesh filename=/home/celdamanufactura/ros2_ws/src/scora-er_14/scora_ind/me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
- link link_4: geometry collision mesh filename=/home/celdamanufactura/ros2_ws/src/scora-er_14/scora_ind/me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; visual mesh filename=/home/celdamanufactura/ros2_ws/src/scora-er_14/scora_ind/me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
- link link_top: geometry collision mesh filename=/home/celdamanufactura/ros2_ws/src/scora-er_14/scora_ind/me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; visual mesh filename=/home/celdamanufactura/ros2_ws/src/scora-er_14/scora_ind/me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
